Commit message: Updated with demo stuff

File: iiwa_tool/iiwa_tool_description/urdf/iiwa_tool.urdf.xacro (robot description, xacro)
@@ -38,6 +38,6 @@
   <!-- Tool properties -->
   <property name="tool_mass" value="0.200" />
-  <property name="tool_joint_offset" value="0.00 0.00 0.00" />
-  <property name="tool_link_offset" value="0.00 0.00 0.1275" />
+  <!-- <property name="tool_joint_offset" value="0.00 0.00 0.00" /> -->
+  <!-- <property name="tool_link_offset" value="0.00 0.00 0.1275" /> -->
   <!--  Here we define a dummy joint between the tip of the iiwa7 and the base of the tool.
   There is no offset between the two, that means the tool is attached at the robot flange. -->
@@ -45,5 +45,5 @@
     <parent link="iiwa_link_ee" />
     <child link = "tool_link" />
-    <origin xyz="${tool_joint_offset}" rpy="0 ${PI/2.0} 0" />
+    <origin xyz="0.00 0.00 0.00" rpy="0 ${PI/2.0} 0" />
   </joint>
   <!-- Here we define the geometry of the tool. We designed the tool ourselves, so we have a mesh file that represents it.
@@ -71,5 +71,5 @@
     <parent link="tool_link" />
     <child link = "tool_link_ee" />
-    <origin xyz="${tool_link_offset}" rpy="0 0 0" />
+    <origin xyz="0.00 0.00 0.1275" rpy="0 0 0" />
   </joint>
   <!--  The TCP frame is here defined -->
